Commit message: update

File: racecar_description/urdf/racecar.xacro (robot description, xacro)
@@ -11,5 +11,5 @@
   </link>
   <joint name="base_link_joint" type="fixed">
-    <origin xyz="0 0 0.05" rpy="0 0 0" />
+    <origin xyz="0 0 0.0" rpy="0 0 0" />
     <parent link="base_link" />
     <child link="chassis" />
@@ -39,5 +39,5 @@
   </link>
   <joint name="left_rear_wheel_joint" type="continuous">
-    <origin xyz="0 0.1 0" rpy="1.5708 0 0" />
+    <origin xyz="0 0.09 0" rpy="1.5708 0 0" />
     <parent link="chassis" />
     <child link="left_rear_wheel" />
@@ -60,5 +60,5 @@
   </link>
   <joint name="right_rear_wheel_joint" type="continuous">
-    <origin xyz="0 -0.1 0" rpy="1.5708 0 0" />
+    <origin xyz="0 -0.09 0" rpy="1.5708 0 0" />
     <parent link="chassis" />
     <child link="right_rear_wheel" />
@@ -78,5 +78,5 @@
   </link>
   <joint name="left_steering_hinge_joint" type="revolute">
-    <origin xyz="0.325 0.1 0" rpy="0 1.5708 0" />
+    <origin xyz="0.332 0.09 0" rpy="0 1.5708 0" />
     <parent link="chassis" />
     <child link="left_steering_hinge" />
@@ -96,5 +96,5 @@
   </link>
   <joint name="right_steering_hinge_joint" type="continuous">
-    <origin xyz="0.325 -0.1 0" rpy="0 1.5708 0" />
+    <origin xyz="0.332 -0.09 0" rpy="0 1.5708 0" />
     <parent link="chassis" />
     <child link="right_steering_hinge" />
@@ -165,5 +165,5 @@
   </link>
   <joint name="hokuyo_joint" type="fixed">
-    <origin xyz="0.265 0.0 0.075" rpy="0 0 0"/>
+    <origin xyz="0.262 0.0 0.192" rpy="0 0 0"/>
     <parent link="chassis" />
     <child link="laser" />
@@ -192,5 +192,5 @@
   </link>
   <joint name="zed_camera_joint" type="fixed">
-    <origin xyz="0.390 0 0.04" rpy="0 0 0"/>
+    <origin xyz="0.352 0 0.158" rpy="0 0 0"/>
     <parent link="chassis"/>
     <child link="zed_camera_link"/>
